Commit message: DOCS: Se creo una nueva carpeta con imagenes de la practica, se agrego el arcivo de la practica y se hicieron modificaciones en el archivo .urdf para velo en Rviz

File: Practica1/Robot_p1.urdf (robot description, URDF)
Before this commit: robot rrp_robot, 10 links, 8 joints
Joints:
- added joint Quieta: type fixed, parent AzulClaro, child cafe_eslabon, origin xyz=0 -0.3 -0.15 rpy=1.57 0 0, limit lower=0 upper=0 effort=0 velocity=0
- joint Prismatica: axis (none) -> 0 1 0; child cafe_eslabon -> Dedo; limit (none) -> lower=-0.02 upper=0.2 effort=3.0 velocity=0.1; origin xyz=0 -0.3 -0.15 rpy=1.57 0 0 -> xyz=0 -0.3 -0.4 rpy=1.57 0 0; type fixed -> prismatic
- joint shoulder_joint: limit (none) -> lower=0 upper=0 effort=0 velocity=0
- joint world_joint: limit (none) -> lower=0 upper=0 effort=0 velocity=0
- joint x_joint: limit (none) -> lower=0 upper=0 effort=0 velocity=0
- joint y_joint: limit (none) -> lower=0 upper=0 effort=0 velocity=0
- joint z_joint: limit (none) -> lower=0 upper=0 effort=0 velocity=0
